Commit message: v2

File: test_robot.urdf (robot description, URDF)
Before this commit: robot test_robot, 2 links, 1 joints
Links:
- removed link back_left_upperleg
- added link back_left_leg; collision mesh filename=back_left_leg.stl scale=0.001 0.001 0.001; visual mesh filename=back_left_leg.stl scale=0.001 0.001 0.001
- added link back_right_leg; collision mesh filename=back_right_leg.stl scale=0.001 0.001 0.001; visual mesh filename=back_right_leg.stl scale=0.001 0.001 0.001
- added link front_left_leg; collision mesh filename=front_left_leg.stl scale=0.001 0.001 0.001; visual mesh filename=front_left_leg.stl scale=0.001 0.001 0.001
- added link front_right_leg, mass 0.310908; collision mesh filename=front_right_leg.stl scale=0.001 0.001 0.001; visual mesh filename=front_right_leg.stl scale=0.001 0.001 0.001
- link base: geometry collision mesh filename=base.stl scale=0.001 0.001 0.001; visual mesh filename=base.stl scale=0.001 0.001 0.001
Joints:
- added joint joint2: type fixed, parent base, child back_right_leg, origin xyz=0 0 0 rpy=0 0 0
- added joint joint3: type fixed, parent base, child front_left_leg, origin xyz=0 0 0 rpy=0 0 0
- added joint joint4: type fixed, parent base, child back_left_leg, origin xyz=0 0 0 rpy=0 0 0
- joint joint1: axis 1 0 0 -> (none); child back_left_upperleg -> front_right_leg; limit lower=-1.57 upper=1.57 effort=10 velocity=100.0 -> (none); origin xyz=-0.153792 -0.034703 0.302 rpy=0 0 0 -> xyz=0 0 0 rpy=0 0 0; type revolute -> fixed

File: test_robot2.urdf (robot description, URDF)
Before this commit: robot test_robot2, 1 links, 0 joints
Links:
- removed link back_left_upperleg
- added link back_left_leg; collision mesh filename=back_left_leg.stl scale=0.001 0.001 0.001; visual mesh filename=back_left_leg.stl scale=0.001 0.001 0.001
- added link back_right_leg; collision mesh filename=back_right_leg.stl scale=0.001 0.001 0.001; visual mesh filename=back_right_leg.stl scale=0.001 0.001 0.001
- added link base, mass 1.15689; collision mesh filename=base.stl scale=0.001 0.001 0.001; visual mesh filename=base.stl scale=0.001 0.001 0.001
- added link front_left_leg; collision mesh filename=front_left_leg.stl scale=0.001 0.001 0.001; visual mesh filename=front_left_leg.stl scale=0.001 0.001 0.001
- added link front_right_leg; collision mesh filename=front_right_leg.stl scale=0.001 0.001 0.001; visual mesh filename=front_right_leg.stl scale=0.001 0.001 0.001
Joints:
- added joint joint1: type revolute, parent base, child front_right_leg, origin xyz=0 0 0 rpy=0 0 0, axis 0 0 1, limit lower=-1.57 upper=1.57 effort=10 velocity=1.0
- added joint joint2: type revolute, parent base, child back_right_leg, origin xyz=0 0 0 rpy=0 0 0, axis 0 0 1, limit lower=-1.57 upper=1.57 effort=10 velocity=1.0
- added joint joint3: type revolute, parent base, child front_left_leg, origin xyz=0 0 0 rpy=0 0 0, axis 0 0 1, limit lower=-1.57 upper=1.57 effort=10 velocity=1.0
- added joint joint4: type revolute, parent base, child back_left_leg, origin xyz=0 0 0 rpy=0 0 0, axis 0 0s 1, limit lower=-1.57 upper=1.57 effort=10 velocity=1.0
