Commit message: comi

File: test_robot2.urdf (robot description, URDF)
Before this commit: robot test_robot, 5 links, 4 joints
Links:
- link base: mass 1.15689 -> 111111.15689
Joints:
- joint joint1: limit lower=-1.57 upper=1.57 effort=10 velocity=1.0 -> lower=-3.14 upper=3.14 effort=10 velocity=10.0; origin xyz=0 0 0 rpy=0 0 0 -> xyz=-0.01221 -0.04413 -0.09471 rpy=0 0 0
